File: Accumulation_Control_PCB.kicad_pcb (KiCad board)
At the start: 4 copper layers, 237.7 x 87.4 mm, 389 parts, among them U10 RSCD06D3, U11 PC817, U12 PC817, U13 RSCD06D3, U14 PC817, U15 PC817, U16 RSCD06D3, U17 PC817, U18 PC817, U19 RSCD06D3, U20 PC817, U21 PC817, U22 RSCD06D3, U23 PC817, U24 PC817, U25 RSCD06D3, U26 PC817, U27 PC817, U28 RSCD06D3, U29 PC817, U30 PC817, U7 PC817, U8 RSCD06D3, U9 PC817

Commit message: VER1.0: разместил все 8 каналов управления
Parts:
- removed C35, C91: 100n, Capacitor_SMD:C_0805_2012Metric_Pad1.18x1.45mm_HandSolder
- removed C36, C38, C54, C62: 56p, Capacitor_SMD:C_0805_2012Metric_Pad1.18x1.45mm_HandSolder
- removed C37, C60: 0.27u, Capacitor_SMD:C_0805_2012Metric_Pad1.18x1.45mm_HandSolder
- removed C39, C41, C52, C53, C63: 2.2u, Capacitor_SMD:C_0805_2012Metric_Pad1.18x1.45mm_HandSolder
- removed C40, C42, C64: 0.1u, Capacitor_SMD:C_0805_2012Metric_Pad1.18x1.45mm_HandSolder
- removed C43: 22u, Capacitor_SMD:C_0805_2012Metric_Pad1.18x1.45mm_HandSolder
- removed C45: 330u, Capacitor_SMD:C_0805_2012Metric_Pad1.18x1.45mm_HandSolder
- removed C46: 22u, Capacitor_SMD:C_1210_3225Metric_Pad1.33x2.70mm_HandSolder
- removed C58: 10u, Capacitor_SMD:C_0805_2012Metric_Pad1.18x1.45mm_HandSolder
- removed C61: 100u, Capacitor_SMD:C_0805_2012Metric_Pad1.18x1.45mm_HandSolder
- removed C90: 1u, Capacitor_SMD:C_0805_2012Metric_Pad1.18x1.45mm_HandSolder
- removed D10: ~, MORNSUN:K78xx-1000R3
- removed D15, D6: ~, Package_TO_SOT_SMD:SOT-23
- removed D16, D7: ~, Package_SO:SOIC-8_7.5x5.85mm_P1.27mm
- removed D9: ~, LED_SMD:LED_0805_2012Metric
- removed J4, J5: ~, Connector_My:Mini-Fit_01x02_Vertical
- removed R23, R24, R25, R28, R41, R42, R45: 2M, Resistor_SMD:R_1206_3216Metric
- removed R26, R30, R33, R34, R43, R47, R50: 1k, Resistor_SMD:R_0805_2012Metric_Pad1.20x1.40mm_HandSolder
- removed R27, R31, R44, R48: 16k, Resistor_SMD:R_1206_3216Metric
- removed R29, R46: 120, Resistor_SMD:R_0805_2012Metric_Pad1.20x1.40mm_HandSolder
- removed R32, R49: 49.9, Resistor_SMD:R_0805_2012Metric_Pad1.20x1.40mm_HandSolder
- removed R38, R51: 750, Resistor_SMD:R_0805_2012Metric_Pad1.20x1.40mm_HandSolder
- removed R53: 100k, Resistor_SMD:R_0805_2012Metric_Pad1.20x1.40mm_HandSolder
- removed U6: ~, Package_TO_SOT_SMD:SOT-23-5
- added C48: 0.1u, Capacitor_SMD:C_1206_3216Metric_Pad1.33x1.80mm_HandSolder, F.Cu at (129.8, 116.3)
- added C49: 10n, Capacitor_SMD:C_0805_2012Metric_Pad1.18x1.45mm_HandSolder, F.Cu at (129.2, 119.5)
- C34: value 56p -> 10u; footprint Capacitor_SMD:C_0805_2012Metric_Pad1.18x1.45mm_HandSolder -> Capacitor_SMD:C_1206_3216Metric_Pad1.33x1.80mm_HandSolder
- C44: footprint Capacitor_SMD:C_1210_3225Metric_Pad1.33x2.70mm_HandSolder -> Capacitor_SMD:C_1206_3216Metric_Pad1.33x1.80mm_HandSolder; moved to F.Cu
- C47: value 0.1u -> 10u
- C50: value 10u -> 2.2u; footprint Capacitor_SMD:C_1206_3216Metric_Pad1.33x1.80mm_HandSolder -> Capacitor_SMD:C_0805_2012Metric_Pad1.18x1.45mm_HandSolder
- C51: value 10n -> 2.2u
- C55: value 100n -> 10u
- C56: value 56p -> 10u
- C57: value 10u -> 1u
- C59: value 1u -> 100u
- C65: value 2.2u -> 1n; footprint Capacitor_SMD:C_0805_2012Metric_Pad1.18x1.45mm_HandSolder -> Capacitor_THT:C_Disc_D7.0mm_W2.5mm_P5.00mm
- C66: value 0.1u -> 10u; footprint Capacitor_SMD:C_0805_2012Metric_Pad1.18x1.45mm_HandSolder -> Capacitor_SMD:C_1206_3216Metric_Pad1.33x1.80mm_HandSolder; moved to B.Cu
- C67: value 1n -> 330u; footprint Capacitor_THT:C_Disc_D7.0mm_W2.5mm_P5.00mm -> Capacitor_THT:CP_Radial_D10.0mm_P5.00mm
- C69: value 330u -> 10u; footprint Capacitor_THT:CP_Radial_D10.0mm_P5.00mm -> Capacitor_SMD:C_1206_3216Metric_Pad1.33x1.80mm_HandSolder; moved to B.Cu
- C70: value 10u -> 330u; footprint Capacitor_SMD:C_1206_3216Metric_Pad1.33x1.80mm_HandSolder -> Capacitor_THT:CP_Radial_D10.0mm_P5.00mm; moved to F.Cu
- C71: value 10u -> 1u; footprint Capacitor_SMD:C_1206_3216Metric_Pad1.33x1.80mm_HandSolder -> Capacitor_SMD:C_0805_2012Metric_Pad1.18x1.45mm_HandSolder
- C72: value 330u -> 1n; footprint Capacitor_THT:CP_Radial_D10.0mm_P5.00mm -> Capacitor_THT:C_Disc_D7.0mm_W2.5mm_P5.00mm
- C73, C82, C84, C86, C88: value 1u -> 100n
- C74: value 1n -> 1u; footprint Capacitor_THT:C_Disc_D7.0mm_W2.5mm_P5.00mm -> Capacitor_SMD:C_0805_2012Metric_Pad1.18x1.45mm_HandSolder
- C75, D44, Q11: moved to F.Cu
- C76, C78, C79, C81: value 100n -> 1u
- D12: value ~ -> TD301MCANFD; footprint LED_SMD:LED_0805_2012Metric -> MORNSUN:TD5(3)01MCANFD
- D13: value TD301MCANFD -> ~; footprint MORNSUN:TD5(3)01MCANFD -> LED_SMD:LED_0805_2012Metric
- D19: value URB2405ZP-10WR3 -> ~; footprint MORNSUN:URB_ZP-10WR3 -> LED_SMD:LED_0805_2012Metric
- D21: value ~ -> URB2405ZP-10WR3; footprint LED_SMD:LED_0805_2012Metric -> MORNSUN:URB_ZP-10WR3
- D22: value BZX84C5V1 -> ~; footprint Package_TO_SOT_SMD:SOT-23_Handsoldering -> LED_SMD:LED_0805_2012Metric
- D23: value ~ -> BZX84C5V1; footprint Diode_SMD:D_SMA_Handsoldering -> Package_TO_SOT_SMD:SOT-23_Handsoldering
- D24, D52, D67, D73: footprint Package_TO_SOT_SMD:SOT-23 -> Diode_SMD:D_SMA_Handsoldering
- D26, D34, D50, D54, D68, D71, D77: footprint LED_SMD:LED_0805_2012Metric -> Package_TO_SOT_SMD:SOT-23
- D27, D31, D33, D39, D45, D53, D60, D66: footprint Package_TO_SOT_SMD:SOT-23 -> LED_SMD:LED_0805_2012Metric
- D28, D32, D40, D61, D64, D70, D79: footprint LED_SMD:LED_0805_2012Metric -> Diode_SMD:D_SMA_Handsoldering
- D29, D37, D51, D69, D72: footprint Diode_SMD:D_SMA_Handsoldering -> LED_SMD:LED_0805_2012Metric
- D30, D42, D56, D62, D65: footprint Diode_SMD:D_SMA_Handsoldering -> Package_TO_SOT_SMD:SOT-23
- J12, J21: footprint Connector_Molex:Molex_Mini-Fit_Jr_5566-04A_2x02_P4.20mm_Vertical -> Connector_My:Mini-Fit_01x02_Vertical
- J2, J6: footprint Connector_My:Mini-Fit_01x02_Vertical -> Connector_Molex:Molex_Mini-Fit_Jr_5566-04A_2x02_P4.20mm_Vertical
- L1: value 4.7u -> ~; footprint Inductor_SMD:L_1812_4532Metric_Pad1.30x3.40mm_HandSolder -> Inductor_SMD:L_CommonModeChoke_TDK_ACM2520-2P
- L2: value ~ -> 4.7u; footprint Inductor_SMD:L_CommonModeChoke_Murata_DLW5BTMxxxSQ2x_5x5mm -> Inductor_SMD:L_1812_4532Metric_Pad1.30x3.40mm_HandSolder
- L3: footprint Inductor_SMD:L_CommonModeChoke_TDK_ACM2520-2P -> Inductor_SMD:L_CommonModeChoke_Murata_DLW5BTMxxxSQ2x_5x5mm; moved to B.Cu
- Q10, Q12, Q14, Q16: footprint Package_TO_SOT_SMD:SOT-223 -> Package_TO_SOT_SMD:SOT-23
- Q3, Q5, Q7, Q9: footprint Package_TO_SOT_SMD:SOT-23 -> Package_TO_SOT_SMD:SOT-223
- R100, R61, R64, R82: value 10k -> 8.2k
- R101, R104, R107, R113, R116, R122, R125, R77, R83, R86, R95: value 8.2k -> 10k
- R102, R84: value 10k -> 330
- R103, R112, R121, R76, R85, R94: value 330 -> 8.2k
- R106, R115, R124, R79, R88, R97: value 1k -> 8.2k
- R108, R111, R117, R120, R126, R129: value 10k -> 1k
- R114, R123: value 3.3k -> 1k
- R131: value 59 -> 10k
- R37: value 8.2k -> 59
- R39: value 59 -> 750; moved to B.Cu
- R40: value 2M -> 59; footprint Resistor_SMD:R_1206_3216Metric -> Resistor_SMD:R_0805_2012Metric_Pad1.20x1.40mm_HandSolder
- R52: value 1k -> 750
- R54: value 2.4k -> 8.2k; footprint Resistor_SMD:R_1206_3216Metric_Pad1.30x1.75mm_HandSolder -> Resistor_SMD:R_0805_2012Metric_Pad1.20x1.40mm_HandSolder
- R55: value 1.1k -> 100k
- R56: value 330 -> 2.4k; footprint Resistor_SMD:R_0805_2012Metric_Pad1.20x1.40mm_HandSolder -> Resistor_SMD:R_1206_3216Metric_Pad1.30x1.75mm_HandSolder
- R57: value 8.2k -> 1.1k; moved to B.Cu
- R58: value 3.3k -> 232
- R59: value 10k -> 100
- R60, R66, R90: value 8.2k -> 330
- R62: value 1k -> 10k
- R63, R81, R99: value 8.2k -> 3.3k
- R65: value 330 -> 10k
- R67: value 3.3k -> 8.2k
- R68: value 232 -> 10k
- R69, R75, R93: value 10k -> 3.3k
- R72: value 1k -> 330
- R74: value 100 -> 10k
- R78, R96: value 3.3k -> 330
- U10, U13, U16, U19, U22, U8: value RSCD06D3 -> PC817; footprint OptoDevice:Finder_34.81 -> Package_DIP:DIP-4_W7.62mm
- U23, U24, U26, U27, U29, U30: value PC817 -> RSCD06D3; footprint Package_DIP:DIP-4_W7.62mm -> OptoDevice:Finder_34.81
- U4: value ~ -> LM1117MP-3.3; footprint Package_TO_SOT_SMD:SOT-23-5 -> Package_TO_SOT_SMD:SOT-223-3_TabPin2
- moved R56 766.3 mm to (-337.2, 199.7)
- moved H3 359.1 mm to (534.4, 293.8)
- moved J2 299.1 mm to (176.4, -87.4)
- moved Q9 275.6 mm to (509.1, 169.2), turned to 90 degrees
- moved R58 272.6 mm to (132.8, 220.5)
- moved R59 272.6 mm to (132.8, 223.4)
- moved J6 267.7 mm to (118.9, 118.0), turned to 0 degrees
- moved R130 266.8 mm to (418.8, 284.5), turned to 180 degrees
- moved D79 264.0 mm to (415.5, 293.5), turned to 90 degrees
- moved Q8 257.0 mm to (472.1, 169.2), turned to 90 degrees
- moved J21 248.1 mm to (479.8, 172.5), turned to 180 degrees
- moved H1 231.9 mm to (225.8, 293.8)
- moved D44 219.4 mm to (429.5, 169.2)
- moved U22 211.0 mm to (525.3, 175.4), turned to -90 degrees
- moved C65 210.8 mm to (235.8, 233.8)
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Connections:
- C10 pad 1: VDC_IN_SENSE -> /Voltage_measure_1/VDC_SENSE
- C22 pad 1: GNDPWR -> Net-(D2-GND1)
- C23 pad 2: GNDPWR -> Net-(D2-GND1)
- C34 pad 2: Net-(U4-+) -> +3.3V
- C44 pad 2: +24V -> +5V
- C50 pad 1: +3.3V -> Net-(U5-VCAP_1)
- C51 pad 1: Net-(C51-Pad1) -> Net-(U5-VCAP_2)
- C51 pad 2: GND_CAN -> GND
- C55 pad 1: +3.3V -> Net-(D18-CS)
- C55 pad 2: GND -> GNDPWR
- C56 pad 1: Net-(D16-VIN) -> +24V
- C56 pad 2: GNDPWR -> GND
- C57 pad 1: Net-(D18-CS) -> Net-(D18-Vin)
- C57 pad 2: GNDPWR -> GND
- C59 pad 1: Net-(D18-Vin) -> +3.3VP
- C59 pad 2: GND -> GNDPWR
- C65 pad 1: GND -> Net-(C65-Pad1)
- C65 pad 2: +3.3V -> +5V
- C66 pad 1: +3.3V -> +5V
- C67 pad 2: +5V -> GNDD
- C68 pad 1: +5V -> Net-(C67-Pad1)
- C68 pad 2: GND -> GNDD
- C69 pad 1: Net-(C69-Pad1) -> Net-(C65-Pad1)
- C69 pad 2: GNDD -> Net-(C69-Pad2)
- C70 pad 1: Net-(C69-Pad1) -> Net-(C65-Pad1)
- C70 pad 2: GNDD -> Net-(C69-Pad2)
- C71 pad 1: Net-(C67-Pad1) -> +5.1V
- C71 pad 2: Net-(C71-Pad2) -> GNDD
- C72 pad 1: Net-(C67-Pad1) -> Net-(C69-Pad2)
- C72 pad 2: Net-(C71-Pad2) -> GND
- C73 pad 1: +5.1V -> GNDPWR
- C73 pad 2: GNDD -> +1V0
- C74 pad 1: Net-(C71-Pad2) -> /Relay_Control_1/Relay_FeedBack
- C75 pad 1: Relay_1_ON -> /Relay_Control_2/Relay_FeedBack
- C76 pad 1: Coil_1_CTRL -> /Relay_Control_3/Relay_FeedBack
- C77 pad 1: Relay_2_ON -> /Relay_Control_4/Relay_FeedBack
- C78 pad 1: GNDPWR -> /Relay_Control_5/Relay_FeedBack
- C78 pad 2: +1V0 -> GND
- C79 pad 1: Coil_2_CTRL -> /Relay_Control_6/Relay_FeedBack
- C80 pad 1: Relay_3_ON -> /Relay_Control_7/Relay_FeedBack
- C81 pad 1: Coil_3_CTRL -> /Relay_Control_8/Relay_FeedBack
- C82 pad 1: Relay_4_ON -> /Solenoid_control_1/Coil_1_CTRL
- C83 pad 1: Coil_4_CTRL -> /Solenoid_control_2/Coil_1_CTRL
- C84 pad 1: Relay_5_ON -> /Solenoid_control_3/Coil_1_CTRL
- C85 pad 1: Coil_5_CTRL -> /Solenoid_control_4/Coil_1_CTRL
- C86 pad 1: Relay_6_ON -> /Solenoid_control_5/Coil_1_CTRL
- C87 pad 1: Coil_6_CTRL -> /Solenoid_control_6/Coil_1_CTRL
- C88 pad 1: Relay_7_ON -> /Solenoid_control_7/Coil_1_CTRL
- C89 pad 1: Coil_7_CTRL -> /Solenoid_control_8/Coil_1_CTRL
- C9 pad 2: GNDPWR -> Net-(D2-GND1)
- D1 pad 3: VDC_IN_SENSE -> /Voltage_measure_1/VDC_SENSE
- D12 pad 1: Net-(D12-K) -> CAN1_RXD_MCU
- D12 pad 2: Net-(D12-A) -> CAN1_TXD_MCU
- D13 pad 1: CAN1_RXD_MCU -> Net-(D13-K)
- D13 pad 2: CAN1_TXD_MCU -> Net-(D13-A)
- D19 pad 1: unconnected-(D19-Ctrl-Pad1) -> Net-(D19-K)
- D19 pad 2: Net-(C71-Pad2) -> +24V
- D2 pad 3: GNDPWR -> Net-(D2-GND1)
- D2 pad 4: GNDPWR -> Net-(D2-GND1)
- D21 pad 1: Net-(D21-K) -> unconnected-(D21-Ctrl-Pad1)
- D21 pad 2: +5V -> Net-(C69-Pad2)
- D22 pad 1: +5.1V -> Net-(D22-K)
- D22 pad 2: GNDD -> +5V
- D23 pad 1: +24V -> +5.1V
- D23 pad 2: Net-(D23-A) -> GNDD
- D24 pad 1: GND -> +24V
- D24 pad 2: +3.3V -> Net-(D24-A)
- D25 pad 2: Net-(D25-A) -> +24V
- D26 pad 1: Net-(D26-K) -> GND
- D26 pad 2: +24V -> +3.3V
- D27 pad 1: GND -> Net-(D27-K)
- D27 pad 2: +3.3V -> Net-(D27-A)
- D28 pad 1: Net-(D28-K) -> +24V
- D29 pad 1: Net-(D28-A) -> Net-(D29-K)
- D29 pad 2: GNDD -> +24V
- D30 pad 1: Net-(D30-K) -> GND
- D30 pad 2: Net-(D30-A) -> +3.3V
- D31 pad 1: GND -> Net-(D31-K)
- D31 pad 2: +3.3V -> Net-(D31-A)
- D32 pad 1: Net-(D32-K) -> +24V
- D33 pad 1: GND -> Net-(D33-K)
- D33 pad 2: +3.3V -> +24V
- D34 pad 1: Net-(D34-K) -> GND
- D34 pad 2: +24V -> +3.3V
- D36 pad 1: Net-(D35-A) -> +24V
- D36 pad 2: GNDD -> Net-(D36-A)
- D37 pad 1: +24V -> Net-(D37-K)
- D37 pad 2: Net-(D37-A) -> +24V
- D38 pad 3: Relay_3_ON -> /Relay_Control_4/Relay_FeedBack
- D39 pad 1: GND -> Net-(D39-K)
- D39 pad 2: +3.3V -> Net-(D39-A)
- D40 pad 1: Net-(D40-K) -> +24V
- D41 pad 2: Net-(D41-A) -> +24V
- D42 pad 1: Net-(D41-A) -> GND
- D42 pad 2: GNDD -> +3.3V
- D43 pad 2: +24V -> Net-(D43-A)
- D45 pad 1: GND -> Net-(D45-K)
- D45 pad 2: +3.3V -> +24V
- D46 pad 3: Coil_4_CTRL -> /Relay_Control_6/Relay_FeedBack
- D48 pad 1: Net-(D47-A) -> +24V
- D48 pad 2: GNDD -> Net-(D48-A)
- D50 pad 1: Net-(D50-K) -> GND
- D50 pad 2: Net-(D50-A) -> +3.3V
- D51 pad 1: +24V -> Net-(D51-K)
- D52 pad 1: GND -> +24V
- D52 pad 2: +3.3V -> Net-(D52-A)
- D53 pad 1: GND -> Net-(D53-K)
- D53 pad 2: +3.3V -> +24V
- D54 pad 1: Net-(D54-K) -> GND
- D54 pad 2: Net-(D54-A) -> +3.3V
- D56 pad 1: Net-(D55-A) -> GND
- D56 pad 2: GNDD -> +3.3V
- D57 pad 2: +24V -> Net-(D57-A)
- D58 pad 1: Net-(D58-K) -> Net-(D57-A)
- D58 pad 2: Net-(D58-A) -> GNDD
- D59 pad 3: Relay_6_ON -> /Solenoid_control_2/Coil_1_CTRL
- D60 pad 1: GND -> Net-(D60-K)
- D60 pad 2: +3.3V -> Net-(D60-A)
- D61 pad 1: Net-(D61-K) -> Net-(D60-A)
- D61 pad 2: Net-(D61-A) -> GNDD
- D62 pad 1: Net-(D61-A) -> GND
- D62 pad 2: GNDD -> +3.3V
- D64 pad 1: Net-(D64-K) -> Net-(D63-A)
- D64 pad 2: +24V -> GNDD
- D65 pad 1: +24V -> GND
- D65 pad 2: Net-(D65-A) -> +3.3V
- D66 pad 1: GND -> Net-(D66-K)
- D66 pad 2: +3.3V -> Net-(D66-A)
- D67 pad 1: GND -> Net-(D66-A)
- D67 pad 2: +3.3V -> GNDD
- D68 pad 1: Net-(D68-K) -> GND
- D68 pad 2: Net-(D68-A) -> +3.3V
- D69 pad 1: Net-(D68-A) -> Net-(D69-K)
- D69 pad 2: GNDD -> Net-(D69-A)
- D70 pad 1: Net-(D70-K) -> Net-(D69-A)
- D70 pad 2: Net-(D70-A) -> GNDD
- D71 pad 1: Net-(D71-K) -> GND
- D71 pad 2: +24V -> +3.3V
- D72 pad 1: +24V -> Net-(D72-K)
- D73 pad 1: GND -> Net-(D72-A)
- D73 pad 2: +3.3V -> GNDD
- D74 pad 3: Relay_8_ON -> /Solenoid_control_7/Coil_1_CTRL
- D77 pad 1: Net-(D77-K) -> GND
- D77 pad 2: Net-(D77-A) -> +3.3V
- D78 pad 2: +24V -> Net-(D78-A)
- D79 pad 1: Net-(D79-K) -> Net-(D78-A)
- D79 pad 2: +24V -> GNDD
- J10 pad 1: GNDD -> Net-(D28-A)
- J10 pad 2: Net-(D41-A) -> +24V
- J11 pad 1: Net-(D44-A) -> Net-(D31-A)
- J12 pad 1: Crrent_Out -> Net-(D32-A)
- J12 pad 2: GND -> +24V
- J13 pad 1: Net-(D50-A) -> Net-(D35-A)
- J14 pad 1: GNDD -> Net-(D36-A)
- J14 pad 2: Net-(D47-A) -> +24V
- J15 pad 1: VDC -> Net-(D39-A)
- J15 pad 2: VDC -> +24V
- J16 pad 1: VDC_OUT1 -> Net-(D40-A)
- J16 pad 2: VDC_OUT1 -> +24V
- J17 pad 1: Net-(D51-A) -> Net-(D43-A)
- J18 pad 1: VDC_OUT2 -> Net-(D44-A)
- J18 pad 2: VDC_OUT2 -> +24V
- J19 pad 1: Net-(D54-A) -> Net-(D47-A)
- J2 pad 1: Net-(D23-A) -> Crrent_Out
- J2 pad 2: +24V -> GND
- J20 pad 1: GNDD -> Net-(D48-A)
- J20 pad 2: Net-(D55-A) -> +24V
- J21 pad 1: CANL -> Net-(D51-A)
- J21 pad 2: CANH -> +24V
- J22 pad 1: GNDPWR -> Net-(D52-A)
- J22 pad 2: GNDPWR -> +24V
- J23 pad 1: Net-(D58-A) -> Net-(D55-A)
- J23 pad 2: Net-(D58-K) -> +24V
- J24 pad 1: Net-(D63-A) -> GNDD
- J24 pad 2: +24V -> Net-(D57-A)
- J25 pad 2: Net-(D61-A) -> Net-(D60-A)
- J26 pad 1: Net-(D65-A) -> GNDD
- J26 pad 2: +24V -> Net-(D63-A)
- J27 pad 1: Net-(D70-A) -> GNDD
- J27 pad 2: +24V -> Net-(D66-A)
- J28 pad 2: Net-(D68-A) -> Net-(D69-A)
- J29 pad 1: Net-(D72-A) -> GNDD
- J29 pad 2: +24V -> Net-(D72-A)
- J3 pad 1: Net-(D25-A) -> Net-(J3-Pin_1)
- J3 pad 2: +24V -> Net-(J3-Pin_1)
- J30 pad 1: Net-(D77-A) -> GNDD
- J30 pad 2: +24V -> Net-(D75-A)
- J31 pad 2: Net-(D75-A) -> Net-(D78-A)
- J6 pad 1: Net-(D32-A) -> CANL
- J6 pad 2: +24V -> CANH
- J7 pad 1: GNDD -> Net-(D2-GND1)
- J7 pad 2: Net-(D35-A) -> Net-(D2-GND1)
- J8 pad 1: Net-(D37-A) -> Net-(D24-A)
- J9 pad 1: Net-(D40-A) -> Net-(D27-A)
- L1 pad 1: +24V -> Net-(D12-CANH)
- L1 pad 2: Net-(D18-Vin) -> Net-(D12-CANL)
- L2 pad 1: Net-(C69-Pad1) -> +24V
- L2 pad 2: Net-(C67-Pad1) -> Net-(D18-Vin)
- L3 pad 1: Net-(D13-CANH) -> Net-(C67-Pad1)
- L3 pad 2: Net-(D13-CANL) -> Net-(C65-Pad1)
- L3 pad 3: CANL -> Net-(C69-Pad2)
- L3 pad 4: CANH -> GNDD
- Q10 pad 2: Net-(D51-A) -> GND
- Q10 pad 3: GNDD -> Net-(Q10-D)
- Q12 pad 2: Net-(D58-A) -> GND
- Q12 pad 3: GNDD -> Net-(Q12-D)
- Q14 pad 2: Net-(D65-A) -> GND
- Q14 pad 3: GNDD -> Net-(Q14-D)
- Q16 pad 2: Net-(D72-A) -> GND
- Q16 pad 3: GNDD -> Net-(Q16-D)
- Q2 pad 2: Net-(D23-A) -> Net-(D24-A)
- Q3 pad 2: GND -> Net-(D28-A)
- Q3 pad 3: Net-(Q3-D) -> GNDD
- Q4 pad 2: Net-(D30-A) -> Net-(D32-A)
- Q5 pad 2: GND -> Net-(D36-A)
- Q5 pad 3: Net-(Q5-D) -> GNDD
- Q6 pad 2: Net-(D37-A) -> Net-(D40-A)
- Q7 pad 2: GND -> Net-(D44-A)
- Q7 pad 3: Net-(Q7-D) -> GNDD
- Q8 pad 2: Net-(D44-A) -> Net-(D48-A)
- Q9 pad 2: GND -> Net-(D52-A)
- Q9 pad 3: Net-(Q9-D) -> GNDD
- R1 pad 2: VDC -> Net-(J3-Pin_1)
- R10 pad 2: VDC_IN_SENSE -> /Voltage_measure_1/VDC_SENSE
- R100 pad 1: Relay_5_ON -> Net-(D51-K)
- R100 pad 2: GND -> GNDD
- R101 pad 1: Net-(D55-K) -> /Relay_Control_7/Relay_FeedBack
- R101 pad 2: GNDD -> GND
- R102 pad 1: GND -> /Relay_Control_8/Relay_CTRL
- R102 pad 2: Net-(Q11-G) -> Net-(R102-Pad2)
- R103 pad 1: Relay_6 -> Net-(D53-K)
- R103 pad 2: Net-(R103-Pad2) -> Net-(D52-A)
- R104 pad 1: Net-(D64-K) -> GNDD
- R104 pad 2: Net-(D58-A) -> Net-(Q9-G)
- R105 pad 2: Net-(D63-A) -> Net-(D55-A)
- R106 pad 1: Coil_6_CTRL -> Net-(D55-K)
- R106 pad 2: Net-(Q13-G) -> GNDD
- R107 pad 1: Net-(D61-K) -> /Relay_Control_8/Relay_FeedBack
- R107 pad 2: GNDD -> GND
- R108 pad 1: GNDD -> /Solenoid_control_1/Coil_1_CTRL
- R108 pad 2: Net-(Q12-G) -> Net-(Q10-G)
- R109 pad 1: Net-(D63-K) -> Net-(D57-K)
- R110 pad 1: Relay_6_ON -> GND
- R110 pad 2: GND -> Net-(Q10-G)
- R111 pad 1: GND -> /Solenoid_control_2/Coil_1_CTRL
- R111 pad 2: Net-(Q13-G) -> Net-(Q11-G)
- R112 pad 1: Relay_8 -> Net-(D60-K)
- R112 pad 2: Net-(R112-Pad2) -> GNDD
- R113 pad 1: Net-(D71-K) -> GND
- R113 pad 2: Net-(D65-A) -> Net-(Q11-G)
- R114 pad 1: Net-(R114-Pad1) -> /Solenoid_control_3/Coil_1_CTRL
- R114 pad 2: Net-(D70-A) -> Net-(Q12-G)
- R115 pad 1: Coil_7_CTRL -> Net-(D63-K)
- R115 pad 2: Net-(Q15-G) -> GNDD
- R116 pad 1: Net-(D68-K) -> GND
- R116 pad 2: GNDD -> Net-(Q12-G)
- R117 pad 1: GNDD -> /Solenoid_control_4/Coil_1_CTRL
- R117 pad 2: Net-(Q14-G) -> Net-(Q13-G)
- R118 pad 1: Net-(D70-K) -> Net-(D66-K)
- R119 pad 1: Relay_7_ON -> GND
- R119 pad 2: GND -> Net-(Q13-G)
- R120 pad 1: GND -> /Solenoid_control_5/Coil_1_CTRL
- R120 pad 2: Net-(Q15-G) -> Net-(Q14-G)
- R121 pad 1: Relay_1 -> Net-(D69-K)
- R121 pad 2: Net-(R121-Pad2) -> GNDD
- R122 pad 1: Net-(D78-K) -> GND
- R122 pad 2: Net-(D72-A) -> Net-(Q14-G)
- R123 pad 1: Net-(R123-Pad1) -> /Solenoid_control_6/Coil_1_CTRL
- R123 pad 2: Net-(D77-A) -> Net-(Q15-G)
- R124 pad 1: Coil_8_CTRL -> Net-(D72-K)
- R124 pad 2: Net-(Q17-G) -> GNDD
- R125 pad 1: Net-(D75-K) -> GND
- R125 pad 2: GNDD -> Net-(Q15-G)
- R126 pad 1: GNDD -> /Solenoid_control_7/Coil_1_CTRL
- R127 pad 1: Net-(D77-K) -> Net-(D75-K)
- R128 pad 1: Relay_8_ON -> GND
- R128 pad 2: GND -> Net-(Q16-G)
- R129 pad 1: GND -> /Solenoid_control_8/Coil_1_CTRL
- R130 pad 1: Net-(D79-K) -> Net-(D78-K)
- R131 pad 1: Net-(C51-Pad1) -> GND
- R131 pad 2: Net-(D13-CANH) -> Net-(Q17-G)
- R36 pad 1: Net-(D12-K) -> Net-(D13-K)
- R37 pad 1: Net-(D9-K) -> Net-(C49-Pad1)
- R37 pad 2: GND -> Net-(D12-CANH)
- R39 pad 1: Net-(D13-CANL) -> Net-(D11-K)
- R39 pad 2: Net-(C51-Pad1) -> GND
- R40 pad 1: Net-(R40-Pad1) -> Net-(D12-CANL)
- R40 pad 2: VDC_OUT2 -> Net-(C49-Pad1)
- R52 pad 1: Net-(U6--) -> Net-(D17-K)
- R52 pad 2: Net-(C62-Pad2) -> GNDPWR
- R54 pad 1: +5.1V -> Net-(D19-K)
- R54 pad 2: +24V -> GNDD
- R55 pad 1: Net-(D21-K) -> Net-(D20-K)
- R55 pad 2: GND -> +24V
- R56 pad 1: Relay_1 -> +5.1V
- R56 pad 2: Net-(R56-Pad2) -> +24V
- R57 pad 1: Net-(D26-K) -> Net-(D22-K)
- R57 pad 2: Net-(D23-A) -> GND
- R58 pad 1: Net-(R58-Pad1) -> +3.3VP
- R58 pad 2: Net-(D25-A) -> +1V0
- R59 pad 1: GNDD -> +1V0
- R59 pad 2: Net-(Q2-G) -> GNDPWR
- R60 pad 1: Net-(D25-K) -> /Relay_Control_1/Relay_CTRL
- R60 pad 2: GNDD -> Net-(R60-Pad2)
- R61 pad 1: Relay_1_ON -> Net-(D25-K)
- R61 pad 2: GND -> Net-(D24-A)
- R62 pad 1: Coil_1_CTRL -> GNDD
- R62 pad 2: Net-(Q3-G) -> Net-(Q2-G)
- R63 pad 1: Net-(D28-K) -> Net-(R63-Pad1)
- R63 pad 2: GNDD -> Net-(D27-A)
- R64 pad 1: GND -> Net-(D27-K)
- R64 pad 2: Net-(Q3-G) -> GNDD
- R65 pad 1: Relay_2 -> /Relay_Control_1/Relay_FeedBack
- R65 pad 2: Net-(R65-Pad2) -> GND
- R66 pad 1: Net-(D34-K) -> /Relay_Control_2/Relay_CTRL
- R66 pad 2: Net-(D30-A) -> Net-(R66-Pad2)
- R67 pad 1: Net-(R67-Pad1) -> Net-(D29-K)
- R67 pad 2: Net-(D32-A) -> Net-(D28-A)
- R68 pad 1: +3.3VP -> GNDD
- R68 pad 2: +1V0 -> Net-(Q3-G)
- R69 pad 1: GNDD -> Net-(R69-Pad1)
- R69 pad 2: Net-(Q4-G) -> Net-(D31-A)
- R70 pad 1: Net-(D32-K) -> Net-(D31-K)
- R71 pad 1: Relay_2_ON -> /Relay_Control_2/Relay_FeedBack
- R72 pad 1: Coil_2_CTRL -> /Relay_Control_3/Relay_CTRL
- R72 pad 2: Net-(Q5-G) -> Net-(R72-Pad2)
- R73 pad 1: Net-(D35-K) -> Net-(D33-K)
- R73 pad 2: GNDD -> Net-(D32-A)
- R74 pad 1: +1V0 -> GNDD
- R74 pad 2: GNDPWR -> Net-(Q4-G)
- R75 pad 1: GND -> Net-(R75-Pad1)
- R75 pad 2: Net-(Q5-G) -> Net-(D35-A)
- R76 pad 1: Relay_3 -> Net-(D35-K)
- R76 pad 2: Net-(R76-Pad2) -> GNDD
- R77 pad 1: Net-(D43-K) -> /Relay_Control_3/Relay_FeedBack
- R77 pad 2: Net-(D37-A) -> GND
- R78 pad 1: Net-(R78-Pad1) -> /Relay_Control_4/Relay_CTRL
- R78 pad 2: Net-(D40-A) -> Net-(R78-Pad2)
- R79 pad 1: Coil_3_CTRL -> Net-(D37-K)
- R79 pad 2: Net-(Q7-G) -> Net-(D36-A)
- R80 pad 2: Net-(Q6-G) -> Net-(Q5-G)
- R81 pad 1: Net-(D40-K) -> Net-(R81-Pad1)
- R81 pad 2: GNDD -> Net-(D39-A)
- R82 pad 1: Relay_3_ON -> Net-(D39-K)
- R82 pad 2: GND -> GNDD
- R83 pad 1: Net-(D41-K) -> /Relay_Control_4/Relay_FeedBack
- R83 pad 2: GNDD -> GND
- R84 pad 1: GND -> /Relay_Control_5/Relay_CTRL
- R84 pad 2: Net-(Q7-G) -> Net-(R84-Pad2)
- R85 pad 1: Relay_4 -> Net-(D41-K)
- R85 pad 2: Net-(R85-Pad2) -> Net-(D40-A)
- R86 pad 1: Net-(D49-K) -> GNDD
- R86 pad 2: Net-(D44-A) -> Net-(Q6-G)
- R87 pad 2: Net-(D50-A) -> Net-(D43-A)
- R88 pad 1: Coil_4_CTRL -> Net-(D43-K)
- R88 pad 2: Net-(Q9-G) -> GNDD
- R89 pad 1: GNDD -> /Relay_Control_5/Relay_FeedBack
- R89 pad 2: Net-(Q8-G) -> GND
- R9 pad 1: GNDPWR -> Net-(D2-GND1)
- R90 pad 1: Net-(D47-K) -> /Relay_Control_6/Relay_CTRL
- R90 pad 2: GNDD -> Net-(R90-Pad2)
- R91 pad 1: Net-(D50-K) -> Net-(D45-K)
- R91 pad 2: GNDD -> Net-(D44-A)
- R92 pad 1: Relay_4_ON -> GNDD
- R92 pad 2: GND -> Net-(Q7-G)
- R93 pad 1: GND -> Net-(R93-Pad1)
- R93 pad 2: Net-(Q9-G) -> Net-(D47-A)
- R94 pad 1: Relay_5 -> Net-(D47-K)
- R94 pad 2: Net-(R94-Pad2) -> GNDD
- R95 pad 1: Net-(D57-K) -> /Relay_Control_6/Relay_FeedBack
- R95 pad 2: Net-(D51-A) -> GND
- R96 pad 1: Net-(R96-Pad1) -> /Relay_Control_7/Relay_CTRL
- R96 pad 2: Net-(D54-A) -> Net-(R96-Pad2)
- R97 pad 1: Coil_5_CTRL -> Net-(D49-K)
- R97 pad 2: Net-(Q11-G) -> Net-(D48-A)
- R98 pad 2: Net-(Q10-G) -> Net-(Q8-G)
- R99 pad 1: Net-(D54-K) -> Net-(R99-Pad1)
- R99 pad 2: GNDD -> Net-(D51-A)
- U11 pad 1: Net-(R65-Pad2) -> Net-(R72-Pad2)
- U12 pad 1: Net-(R67-Pad1) -> Net-(R75-Pad1)
- U12 pad 3: Relay_2_ON -> /Relay_Control_3/Relay_FeedBack
- U14 pad 1: Net-(R76-Pad2) -> Net-(R81-Pad1)
- U14 pad 2: GND -> GNDD
- U14 pad 3: Net-(Q6-G) -> /Relay_Control_4/Relay_FeedBack
- U14 pad 4: +5.1V -> +3.3V
- U15 pad 1: Net-(R78-Pad1) -> Net-(R84-Pad2)
- U15 pad 2: GNDD -> GND
- U15 pad 3: Relay_3_ON -> Net-(Q6-G)
- U15 pad 4: +3.3V -> +5.1V
- U17 pad 1: Net-(R85-Pad2) -> Net-(R90-Pad2)
- U17 pad 3: Net-(Q8-G) -> Net-(Q7-G)
- U18 pad 1: Net-(R87-Pad1) -> Net-(R93-Pad1)
- U18 pad 3: Relay_4_ON -> /Relay_Control_6/Relay_FeedBack
- U20 pad 1: Net-(R94-Pad2) -> Net-(R99-Pad1)
- U20 pad 2: GND -> GNDD
- U20 pad 3: Net-(Q10-G) -> /Relay_Control_7/Relay_FeedBack
- U20 pad 4: +5.1V -> +3.3V
- U21 pad 1: Net-(R96-Pad1) -> Net-(R102-Pad2)
- U21 pad 2: GNDD -> GND
- U21 pad 3: Relay_5_ON -> Net-(Q9-G)
- U21 pad 4: +3.3V -> +5.1V
- U25 pad 14: Net-(D68-A) -> Net-(D63-A)
- U25 pad A2: Net-(Q15-D) -> Net-(Q12-D)
- U28 pad 14: Net-(D75-A) -> Net-(D72-A)
- U28 pad A2: Net-(Q17-D) -> Net-(Q15-D)
- U4 pad 1: Net-(U4-+) -> GND
- U4 pad 2: GND -> +3.3V
- U4 pad 3: Net-(U4--) -> +5V
- U5 pad 57: Net-(D12-A) -> Net-(D13-A)
- U7 pad 1: Net-(R56-Pad2) -> Net-(R60-Pad2)
- U9 pad 1: Net-(R58-Pad1) -> Net-(R66-Pad2)
- U9 pad 2: GNDD -> GND
- U9 pad 3: Relay_1_ON -> Net-(Q3-G)
- U9 pad 4: +3.3V -> +5.1V
Routing:
- net (no net): track 435.5 -> 0.00 mm
- net VDC_OUT1_SENSE: track 228.8 -> 0.00 mm
- net GNDD: track 38.2 -> 150.1 mm, vias 6 -> 8
- net GNDPWR: track 90.3 -> 0.00 mm, vias 9 -> 0
- net VDC_IN_SENSE: track 90.1 -> 0.00 mm
- net Net-(Q4-G): track 95.1 -> 5.42 mm
- net VIN_Enable: track 69.8 -> 0.00 mm
- net Precharge_2: track 65.5 -> 0.00 mm
- net +24V: track 78.3 -> 137.1 mm, vias 5 -> 0
- net +24V_SENSE: track 58.1 -> 0.00 mm
- net +3.3V: track 95.0 -> 37.7 mm, vias 25 -> 19
- net CANH: track 51.4 -> 0.00 mm, vias 2 -> 0
- net CANL: track 49.3 -> 0.00 mm
- net -24V: track 44.9 -> 0.00 mm, vias 2 -> 0
- net Net-(D72-A): track 0.00 -> 31.9 mm
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- added copper zone on F.Cu, net GNDD
- removed copper zone on In1.Cu, net +1V0
- removed copper zone on F.Cu, net +24V
- removed copper zone on In1.Cu, net +24V
- removed copper zone on In1.Cu, net +3.3V
- removed copper zone on F.Cu, net +3.3VP
- removed copper zone on In2.Cu, net +3.3VP
- removed copper zone on In2.Cu, net +5V
- removed copper zone on B.Cu, net GNDPWR
- removed copper zone on F.Cu, net GNDPWR
- removed copper zone on F.Cu, net Net-(U6--)
Other:
- board size 237.7 x 87.4 mm -> 319.7 x 137.4 mm
- board text removed: "GNDPWR"
- board text removed: "VDC IN"
- board text removed: "VOUT 1"
- board text removed: "VOUT 2"

Commit message: VER1.0: улучшил и расставил каналы измерения напряжения
Parts:
- removed C11, C8: 100n, Capacitor_SMD:C_0805_2012Metric_Pad1.18x1.45mm_HandSolder
- removed C21: 56p, Capacitor_SMD:C_0805_2012Metric_Pad1.18x1.45mm_HandSolder
- removed D4: ~, Package_TO_SOT_SMD:SOT-23
- removed R12: 14k, Resistor_SMD:R_0805_2012Metric_Pad1.20x1.40mm_HandSolder
- removed R19: 120, Resistor_SMD:R_0805_2012Metric_Pad1.20x1.40mm_HandSolder
- removed R20: 1k, Resistor_SMD:R_0805_2012Metric_Pad1.20x1.40mm_HandSolder
- removed U3: ~, Package_TO_SOT_SMD:SOT-23-5
- added C35: 10u, Capacitor_SMD:C_1206_3216Metric_Pad1.33x1.80mm_HandSolder, B.Cu at (510.0, 212.8)
- added C36: 10u, Capacitor_SMD:C_1206_3216Metric_Pad1.33x1.80mm_HandSolder, F.Cu at (515.3, 218.3)
- added C37: 10u, Capacitor_SMD:C_1206_3216Metric_Pad1.33x1.80mm_HandSolder, B.Cu at (512.8, 204.8)
- added C38: 10u, Capacitor_SMD:C_1206_3216Metric_Pad1.33x1.80mm_HandSolder, B.Cu at (497.3, 196.0)
- added C39: 1u, Capacitor_SMD:C_1206_3216Metric_Pad1.33x1.80mm_HandSolder, B.Cu at (497.3, 205.0)
- added C40: 56p, Capacitor_SMD:C_0805_2012Metric_Pad1.18x1.45mm_HandSolder, F.Cu at (495.8, 260.8)
- added C41: 100n, Capacitor_SMD:C_0805_2012Metric_Pad1.18x1.45mm_HandSolder, B.Cu at (490.8, 255.0)
- added C42: 56p, Capacitor_SMD:C_0805_2012Metric_Pad1.18x1.45mm_HandSolder, F.Cu at (512.8, 254.5)
- added C43: 0.27u, Capacitor_SMD:C_0805_2012Metric_Pad1.18x1.45mm_HandSolder, F.Cu at (487.5, 259.5)
- added C45: 56p, Capacitor_SMD:C_0805_2012Metric_Pad1.18x1.45mm_HandSolder, F.Cu at (495.8, 249.2)
- added C46: 2.2u, Capacitor_SMD:C_0805_2012Metric_Pad1.18x1.45mm_HandSolder, B.Cu at (510.2, 255.0)
- added C52: 0.1u, Capacitor_SMD:C_0805_2012Metric_Pad1.18x1.45mm_HandSolder, B.Cu at (508.0, 255.0)
- added C53: 2.2u, Capacitor_SMD:C_0805_2012Metric_Pad1.18x1.45mm_HandSolder, B.Cu at (502.0, 255.0)
- added C54: 0.1u, Capacitor_SMD:C_0805_2012Metric_Pad1.18x1.45mm_HandSolder, B.Cu at (499.8, 255.0)
- added C58: 0.27u, Capacitor_SMD:C_0805_2012Metric_Pad1.18x1.45mm_HandSolder, F.Cu at (487.5, 279.5)
- added C60: 56p, Capacitor_SMD:C_0805_2012Metric_Pad1.18x1.45mm_HandSolder, F.Cu at (495.8, 269.2)
- added C61: 2.2u, Capacitor_SMD:C_0805_2012Metric_Pad1.18x1.45mm_HandSolder, B.Cu at (510.2, 275.0)
- added C62: 0.1u, Capacitor_SMD:C_0805_2012Metric_Pad1.18x1.45mm_HandSolder, B.Cu at (508.0, 275.0)
- added C63: 2.2u, Capacitor_SMD:C_0805_2012Metric_Pad1.18x1.45mm_HandSolder, B.Cu at (502.0, 275.0)
- added C64: 0.1u, Capacitor_SMD:C_0805_2012Metric_Pad1.18x1.45mm_HandSolder, B.Cu at (499.8, 275.0)
- added D10: TO-3216BC-MYF, LED_SMD:LED_1206_3216Metric_Pad1.42x1.75mm_HandSolder, F.Cu at (524.5, 255.0)
- added D15: ~, Package_SO:SOIC-8_7.5x5.85mm_P1.27mm, F.Cu at (505.0, 255.0)
- added D16: S1M, Diode_SMD:D_SMA_Handsoldering, B.Cu at (522.2, 259.5)
- added D6: TO-3216BC-MYF, LED_SMD:LED_1206_3216Metric_Pad1.42x1.75mm_HandSolder, F.Cu at (524.5, 235.0)
- added D7: S1M, Diode_SMD:D_SMA_Handsoldering, B.Cu at (522.2, 239.5)
- added D80: ~, Package_TO_SOT_SMD:SOT-23, F.Cu at (484.5, 279.5)
- added D81: TO-3216BC-MYF, LED_SMD:LED_1206_3216Metric_Pad1.42x1.75mm_HandSolder, F.Cu at (524.5, 275.0)
- added D82: ~, Package_SO:SOIC-8_7.5x5.85mm_P1.27mm, F.Cu at (505.0, 275.0)
- added D83: S1M, Diode_SMD:D_SMA_Handsoldering, B.Cu at (522.2, 279.5)
- added D9: ~, Package_TO_SOT_SMD:SOT-23, F.Cu at (484.5, 259.5)
- added F1: 0451002.MRL, Fuse_my:SMD_2410, F.Cu at (234.2, 235.2)
- added J32: ~, Connector_My:Mini-Fit_01x02_Vertical, F.Cu at (529.2, 270.5)
- added J33: ~, Connector_My:Mini-Fit_01x02_Vertical, F.Cu at (529.2, 279.5)
- added J34: ~, Connector_Molex:Molex_Mini-Fit_Jr_5566-04A_2x02_P4.20mm_Vertical, F.Cu at (230.5, 202.9)
- added J4: ~, Connector_My:Mini-Fit_01x02_Vertical, F.Cu at (529.2, 250.5)
- added J5: ~, Connector_My:Mini-Fit_01x02_Vertical, F.Cu at (529.2, 259.5)
- added R132: 150k, Resistor_SMD:R_1206_3216Metric, B.Cu at (520.8, 273.5)
- added R133: 16k, Resistor_SMD:R_1206_3216Metric, F.Cu at (523.0, 282.2)
- added R134: 2M, Resistor_SMD:R_1206_3216Metric, F.Cu at (519.2, 277.0)
- added R135: 120, Resistor_SMD:R_0805_2012Metric_Pad1.20x1.40mm_HandSolder, F.Cu at (518.0, 282.2)
- added R136: 1k, Resistor_SMD:R_0805_2012Metric_Pad1.20x1.40mm_HandSolder, F.Cu at (495.8, 276.2)
- added R137: 16k, Resistor_SMD:R_1206_3216Metric, F.Cu at (523.0, 279.5)
- added R138: 49.9, Resistor_SMD:R_0805_2012Metric_Pad1.20x1.40mm_HandSolder, F.Cu at (489.8, 279.5)
- added R139: 1k, Resistor_SMD:R_0805_2012Metric_Pad1.20x1.40mm_HandSolder, F.Cu at (495.8, 273.8)
- added R140: 1k, Resistor_SMD:R_0805_2012Metric_Pad1.20x1.40mm_HandSolder, F.Cu at (495.8, 271.5)
- added R23: 240, Resistor_SMD:R_0805_2012Metric_Pad1.20x1.40mm_HandSolder, F.Cu at (522.0, 214.8)
- added R24: 1k, Resistor_SMD:R_0805_2012Metric_Pad1.20x1.40mm_HandSolder, F.Cu at (522.0, 212.5)
- added R25: 150k, Resistor_SMD:R_1206_3216Metric, B.Cu at (520.8, 233.5)
- added R26: 150k, Resistor_SMD:R_1206_3216Metric, B.Cu at (517.2, 231.5)
- added R27: 150k, Resistor_SMD:R_1206_3216Metric, B.Cu at (520.8, 229.5)
- added R28: 150k, Resistor_SMD:R_1206_3216Metric, B.Cu at (520.8, 249.5)
- added R29: 2M, Resistor_SMD:R_1206_3216Metric, F.Cu at (523.0, 248.8)
- added R30: 2M, Resistor_SMD:R_1206_3216Metric, F.Cu at (519.2, 250.8)
- added R31: 150k, Resistor_SMD:R_1206_3216Metric, B.Cu at (517.2, 251.5)
- added R32: 2M, Resistor_SMD:R_1206_3216Metric, F.Cu at (516.8, 253.8)
- added R33: 1k, Resistor_SMD:R_0805_2012Metric_Pad1.20x1.40mm_HandSolder, F.Cu at (495.8, 258.5)
- added R34: 150k, Resistor_SMD:R_1206_3216Metric, B.Cu at (520.8, 253.5)
- added R38: 16k, Resistor_SMD:R_1206_3216Metric, F.Cu at (523.0, 262.2)
- added R41: 2M, Resistor_SMD:R_1206_3216Metric, F.Cu at (519.2, 257.0)
- added R42: 120, Resistor_SMD:R_0805_2012Metric_Pad1.20x1.40mm_HandSolder, F.Cu at (518.0, 262.2)
- added R43: 1k, Resistor_SMD:R_0805_2012Metric_Pad1.20x1.40mm_HandSolder, F.Cu at (495.8, 256.2)
- added R44: 16k, Resistor_SMD:R_1206_3216Metric, F.Cu at (523.0, 259.5)
- added R45: 49.9, Resistor_SMD:R_0805_2012Metric_Pad1.20x1.40mm_HandSolder, F.Cu at (489.8, 259.5)
- added R46: 1k, Resistor_SMD:R_0805_2012Metric_Pad1.20x1.40mm_HandSolder, F.Cu at (495.8, 253.8)
- added R47: 1k, Resistor_SMD:R_0805_2012Metric_Pad1.20x1.40mm_HandSolder, F.Cu at (495.8, 251.5)
- added R48: 150k, Resistor_SMD:R_1206_3216Metric, B.Cu at (520.8, 269.5)
- added R49: 2M, Resistor_SMD:R_1206_3216Metric, F.Cu at (523.0, 268.8)
- added R50: 2M, Resistor_SMD:R_1206_3216Metric, F.Cu at (519.2, 270.8)
- added R51: 150k, Resistor_SMD:R_1206_3216Metric, B.Cu at (517.2, 271.5)
- added R53: 2M, Resistor_SMD:R_1206_3216Metric, F.Cu at (516.8, 273.8)
- added U31: TLV1117LV33DCYR, Package_TO_SOT_SMD:SOT-223-3_TabPin2, F.Cu at (510.0, 219.8)
- added U32: OPA333xxDBV, Package_TO_SOT_SMD:SOT-23-5, F.Cu at (490.8, 255.0)
- added U33: OPA333xxDBV, Package_TO_SOT_SMD:SOT-23-5, F.Cu at (490.8, 275.0)
- added U6: OPA333xxDBV, Package_TO_SOT_SMD:SOT-23-5, F.Cu at (490.8, 235.0)
- C1, C10, C12, C14, C15, C7, C71, C73, R2, R3: moved to F.Cu
- C16, C17, C18, C19, C23, C24, C25, C27, C28, C29, C32, C33, C48, R52: moved to B.Cu
- C26, C30: value 30p -> 12p
- C55: value 10u -> 56p; moved to F.Cu
- C56: value 10u -> 100n
- C57: value 1u -> 56p
- R58: value 232 -> 1k
- R59: value 100 -> 1k
- U1: value ~ -> TLV431; footprint Package_TO_SOT_SMD:SOT-23-5 -> Package_TO_SOT_SMD:SOT-23
- U2: value ~ -> OPA333xxDBV
- U4: value LM1117MP-3.3 -> TLV1117LV33DCYR
- moved R56 565.1 mm to (227.8, 184.0)
- moved R13 439.3 mm to (495.8, 233.8), turned to 180 degrees
- moved J7 424.8 mm to (529.2, 239.5), turned to 90 degrees
- moved C25 408.4 mm to (499.8, 235.0)
- moved L2 399.1 mm to (499.8, 200.5), turned to 90 degrees
- moved C24 390.0 mm to (502.0, 235.0)
- moved R58 386.5 mm to (519.3, 218.3), turned to 90 degrees
- moved R59 367.2 mm to (495.8, 278.5), turned to 180 degrees
- moved J3 363.6 mm to (529.2, 230.5), turned to 90 degrees
- moved Y1 330.1 mm to (380.0, 250.2), turned to 180 degrees
- moved D8 325.7 mm to (170.2, 193.8)
- moved R11 325.7 mm to (160.0, 193.8)
- moved R15 307.1 mm to (192.0, 196.5)
- moved R18 307.1 mm to (192.0, 201.6)
- moved J2 298.0 mm to (167.2, 210.5)
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Connections:
- C1 pad 2: Net-(U1-+) -> Net-(U6-+)
- C12 pad 1: Net-(U1--) -> Net-(U6--)
- C22 pad 1: Net-(D2-GND1) -> GNDPWR
- C23 pad 2: Net-(D2-GND1) -> GNDPWR
- C55 pad 1: Net-(D18-CS) -> GND
- C55 pad 2: GNDPWR -> Net-(U33-+)
- C56 pad 1: +24V -> +3.3V
- C57 pad 1: Net-(D18-Vin) -> Net-(D82-VIN)
- C57 pad 2: GND -> GNDPWR
- C59 pad 1: +3.3VP -> Net-(D18-+Vo)
- C9 pad 2: Net-(D2-GND1) -> GNDPWR
- D18 pad 6: +3.3VP -> Net-(D18-+Vo)
- D2 pad 3: Net-(D2-GND1) -> GNDPWR
- D2 pad 4: Net-(D2-GND1) -> GNDPWR
- J6 pad 1: CANL -> -24V
- J6 pad 2: CANH -> +24V
- J6 pad 3: +24V -> -24V
- J6 pad 4: -24V -> +24V
- J7 pad 1: Net-(D2-GND1) -> GNDPWR
- J7 pad 2: Net-(D2-GND1) -> GNDPWR
- R13 pad 2: Net-(U1--) -> Net-(U6--)
- R21 pad 1: Net-(U1--) -> Net-(U6--)
- R4 pad 2: Net-(U1-+) -> Net-(U6-+)
- R58 pad 2: +1V0 -> Net-(U1-K)
- R59 pad 1: +1V0 -> GND
- R59 pad 2: GNDPWR -> Net-(U33-+)
- R8 pad 2: Net-(U1-+) -> Net-(U6-+)
- R9 pad 1: Net-(D2-GND1) -> GNDPWR
- U1 pad 1: Net-(U1-+) -> Net-(U1-K)
- U1 pad 2: GND -> Net-(U1-K)
- U1 pad 3: Net-(U1--) -> GNDPWR
- U2 pad 1: Net-(U2-+) -> Net-(U2--)
- U2 pad 3: Net-(U2--) -> Net-(U2-+)
Routing:
- net GNDPWR: track 0.00 -> 67.5 mm, vias 0 -> 3
- net GNDD: track 150.1 -> 98.8 mm, vias 8 -> 0
- net GND: track 102.2 -> 55.9 mm, vias 55 -> 6
- net CAN1_TXD_MCU: track 0.00 -> 22.7 mm
- net Net-(C45-Pad2): track 0.00 -> 21.5 mm
- net Net-(C12-Pad2): track 0.00 -> 21.5 mm
- net Net-(C60-Pad2): track 0.00 -> 21.5 mm
- net Net-(J4-Pin_1): track 0.00 -> 18.5 mm
- net Net-(J32-Pin_1): track 0.00 -> 18.5 mm
- net Net-(J3-Pin_1): track 0.00 -> 18.5 mm
- net CAN1_RXD_MCU: track 0.00 -> 17.6 mm
- net +3.3VP: track 0.00 -> 14.5 mm, vias 0 -> 3
- net +3.3V: track 37.7 -> 23.2 mm, vias 19 -> 6
- net Net-(D2-VIN): track 0.00 -> 12.3 mm
- net Net-(D15-VIN): track 0.00 -> 12.3 mm
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- removed copper zone on B.Cu, net GND
Other:
- board text added: "+24V"
- board text added: "+5V"
- board text removed: "DAC1"
- board text removed: "DAC2"
- board text removed: "GPIO"
- board text removed: "IN/OUT"
