File: Accumulation_Control_PCB.kicad_sch (KiCad schematic)
At the start: 388 parts, among them U10 RSCD06D3, U11 PC817, U12 PC817, U13 RSCD06D3, U14 PC817, U15 PC817, U16 RSCD06D3, U17 PC817, U18 PC817, U19 RSCD06D3, U20 PC817, U21 PC817, U22 RSCD06D3, U23 PC817, U24 PC817, U25 RSCD06D3, U26 PC817, U27 PC817, U28 RSCD06D3, U29 PC817, U30 PC817, U7 PC817, U8 RSCD06D3, U9 PC817

Commit message: VER1.0: разместил все 8 каналов управления
Parts:
- removed C1, C12, C34, C36, C38, C54, C56, C62, C9: 56p, Capacitor_SMD:C_0805_2012Metric_Pad1.18x1.45mm_HandSolder, symbol Device:C
- removed C10, C37, C60: 0.27u, Capacitor_SMD:C_0805_2012Metric_Pad1.18x1.45mm_HandSolder, symbol Device:C
- removed C2, C35, C55: 100n, Capacitor_SMD:C_0805_2012Metric_Pad1.18x1.45mm_HandSolder, symbol Device:C
- removed C22, C24, C39, C41, C63, C65: 2.2u, Capacitor_SMD:C_0805_2012Metric_Pad1.18x1.45mm_HandSolder, symbol Device:C
- removed C23, C25, C40, C42, C64, C66: 0.1u, Capacitor_SMD:C_0805_2012Metric_Pad1.18x1.45mm_HandSolder, symbol Device:C
- removed C43: 22u, Capacitor_Tantalum_SMD:CP_EIA-7343-43_Kemet-X_Pad2.25x2.55mm_HandSolder, symbol Device:C_Polarized_Small
- removed C45: 330u, Capacitor_Tantalum_SMD:CP_EIA-6032-28_Kemet-C_Pad2.25x2.35mm_HandSolder, symbol Device:C_Polarized_Small
- removed C46: 22u, Capacitor_SMD:C_1210_3225Metric_Pad1.33x2.70mm_HandSolder, symbol Device:C_Small
- removed C75, C77, C80, C82, C84, C86, C88, C90: 1u, Capacitor_SMD:C_0805_2012Metric_Pad1.18x1.45mm_HandSolder, symbol Device:C_Small
- removed C76, C79, C81, C83, C85, C87, C89, C91: 100n, Capacitor_SMD:C_0805_2012Metric_Pad1.18x1.45mm_HandSolder, symbol Device:C_Small
- removed D1, D15, D24, D27, D31, D33, D38, D39, D45, D46, D52, D53, D59, D6, D60, D66, D67, D73, D74: ~, Package_TO_SOT_SMD:SOT-23, symbol Device:D_Dual_Series_AKC_Parallel
- removed D10: ~, MORNSUN:K78xx-1000R3, symbol MORNSUN:K78xx-1000R3
- removed D16, D2, D7: ~, Package_SO:SOIC-8_7.5x5.85mm_P1.27mm, symbol NOVSENSE:NSI1311
- removed D23, D29, D30, D36, D37, D42, D44, D48, D51, D56, D58, D62, D65, D69, D72, D76: ~, Diode_SMD:D_SMA_Handsoldering, symbol Device:D_Small
- removed D25, D26, D28, D32, D34, D35, D40, D41, D43, D47, D49, D50, D54, D55, D57, D61, D63, D64, D68, D70, D71, D75, D77, D78, D9: ~, LED_SMD:LED_0805_2012Metric, symbol Device:LED_Small
- removed J10, J11, J13, J14, J15, J16, J17, J18, J19, J2, J20, J22, J23, J24, J25, J26, J27, J28, J29, J3, J30, J31, J4, J5, J6, J7, J8, J9: ~, Connector_My:Mini-Fit_01x02_Vertical, symbol Connector_Generic:Conn_01x02
- removed Q10, Q12, Q14, Q16, Q2, Q4, Q6, Q8: ~, Package_TO_SOT_SMD:SOT-223, symbol Driver_FET:BSP75N
- removed Q11, Q13, Q15, Q17, Q3, Q5, Q7, Q9: ~, Package_TO_SOT_SMD:SOT-23, symbol Transistor_FET:2N7002
- removed R1, R2, R23, R24, R25, R28, R3, R40, R41, R42, R45, R6: 2M, Resistor_SMD:R_1206_3216Metric, symbol Device:R
- removed R10, R32, R49: 49.9, Resistor_SMD:R_0805_2012Metric_Pad1.20x1.40mm_HandSolder, symbol Device:R
- removed R100, R102, R108, R110, R111, R117, R119, R120, R126, R128, R129, R59, R61, R64, R69, R71, R75, R80, R82, R84, R89, R92, R93, R98: 10k, Resistor_SMD:R_0805_2012Metric_Pad1.20x1.40mm_HandSolder, symbol Device:R_Small
- removed R101, R104, R107, R109, R113, R116, R118, R122, R125, R127, R37, R57, R60, R63, R66, R70, R73, R77, R81, R83, R86, R90, R91, R95, R99: 8.2k, Resistor_SMD:R_0805_2012Metric_Pad1.20x1.40mm_HandSolder, symbol Device:R_Small
- removed R103, R112, R121, R56, R65, R76, R85, R94: 330, Resistor_SMD:R_0805_2012Metric_Pad1.20x1.40mm_HandSolder, symbol Device:R_Small
- removed R105, R114, R123, R58, R67, R78, R87, R96: 3.3k, Resistor_SMD:R_0805_2012Metric_Pad1.20x1.40mm_HandSolder, symbol Device:R_Small
- removed R106, R115, R124, R62, R72, R79, R88, R97: 1k, Resistor_SMD:R_0805_2012Metric_Pad1.20x1.40mm_HandSolder, symbol Device:R_Small
- removed R13, R21, R26, R30, R33, R34, R4, R43, R47, R50, R52, R8: 1k, Resistor_SMD:R_0805_2012Metric_Pad1.20x1.40mm_HandSolder, symbol Device:R
- removed R27, R31, R44, R48, R5, R9: 16k, Resistor_SMD:R_1206_3216Metric, symbol Device:R
- removed R29, R46, R7: 120, Resistor_SMD:R_0805_2012Metric_Pad1.20x1.40mm_HandSolder, symbol Device:R
- removed U1, U4, U6: ~, Package_TO_SOT_SMD:SOT-23-5, symbol Amplifier_Operational:LMV321
- removed U10, U13, U16, U19, U22, U25, U28, U8: RSCD06D3, OptoDevice:Finder_34.81, symbol Relay_SolidState:34.81-7048
- removed U11, U12, U14, U15, U17, U18, U20, U21, U23, U24, U26, U27, U29, U30, U7, U9: PC817, Package_DIP:DIP-4_W7.62mm, symbol Isolator:PC817
- added C34: 10u, Capacitor_SMD:C_1206_3216Metric_Pad1.33x1.80mm_HandSolder, symbol Device:C_Small
- added U4: LM1117MP-3.3, Package_TO_SOT_SMD:SOT-223-3_TabPin2, symbol Regulator_Linear:LM1117MP-3.3
- C44: footprint Capacitor_SMD:C_1210_3225Metric_Pad1.33x2.70mm_HandSolder -> Capacitor_SMD:C_1206_3216Metric_Pad1.33x1.80mm_HandSolder
- renumbered C50 to C47, C47 to C48, C51 to C49, C52 to C50, C53 to C51, C57 to C55, C58 to C56, C59 to C57, C61 to C59, C67 to C65, C68 to C66, C69 to C67, C70 to C68, C71 to C69, C72 to C70, C73 to C71, C74 to C72, C78 to C73, D13 to D12, D12 to D13, D79 to D19, D19 to D21, D21 to D22, D22 to D23, J12 to J2, J21 to J6, L3 to L1, L1 to L2, L2 to L3, R131 to R37, R38 to R39, R39 to R40, R51 to R52, R130 to R54, R53 to R55, R54 to R56, R55 to R57, R68 to R58, R74 to R59
Connections:
- net +24V: no longer C44.2
- net +3.3V: now also C34.2, U4.2 (VO)
- net +5V: now also C44.2, U4.3 (VI)
- net GND: now also C34.1, U4.1 (GND)
Other:
- added sheet Relay_Control_1 (Power_relay_control.kicad_sch)
- added sheet Relay_Control_2 (Power_relay_control.kicad_sch)
- added sheet Relay_Control_3 (Power_relay_control.kicad_sch)
- added sheet Relay_Control_4 (Power_relay_control.kicad_sch)
- added sheet Relay_Control_5 (Power_relay_control.kicad_sch)
- added sheet Relay_Control_6 (Power_relay_control.kicad_sch)
- added sheet Relay_Control_7 (Power_relay_control.kicad_sch)
- added sheet Relay_Control_8 (Power_relay_control.kicad_sch)
- added sheet Solenoid_control_1 (Solenoid_control.kicad_sch)
- added sheet Solenoid_control_2 (Solenoid_control.kicad_sch)
- added sheet Solenoid_control_3 (Solenoid_control.kicad_sch)
- added sheet Solenoid_control_4 (Solenoid_control.kicad_sch)
- added sheet Solenoid_control_5 (Solenoid_control.kicad_sch)
- added sheet Solenoid_control_6 (Solenoid_control.kicad_sch)
- added sheet Solenoid_control_7 (Solenoid_control.kicad_sch)
- added sheet Solenoid_control_8 (Solenoid_control.kicad_sch)
- added sheet Voltage_measure_1 (Voltage_measure.kicad_sch)
- note removed: "Измерение высокого входного напряжения"
- note removed: "Измерение высокого выходного напряжения 1"
- note removed: "Измерение высокого выходного напряжения 2"
- note removed: "Индикация замыкания контакторов"
- note removed: "Управление клапанами"
- note removed: "Управление контакторами"
- moved on the sheet: C44

Commit message: VER1.0: улучшил и расставил каналы измерения напряжения
Parts:
- removed C11, C8: 100n, Capacitor_SMD:C_0805_2012Metric_Pad1.18x1.45mm_HandSolder, symbol Device:C_Small
- removed C21: 56p, Capacitor_SMD:C_0805_2012Metric_Pad1.18x1.45mm_HandSolder, symbol Device:C_Small
- removed C55: 10u, Capacitor_Tantalum_SMD:CP_EIA-3528-21_Kemet-B_Pad1.50x2.35mm_HandSolder, symbol Device:C_Polarized
- removed C56: 10u, Capacitor_Tantalum_SMD:CP_EIA-7360-38_Kemet-E_Pad2.25x4.25mm_HandSolder, symbol Device:C_Polarized
- removed C57: 1u, Capacitor_Tantalum_SMD:CP_EIA-6032-28_Kemet-C_Pad2.25x2.35mm_HandSolder, symbol Device:C_Polarized
- removed D4: ~, Package_TO_SOT_SMD:SOT-23, symbol Device:D_Dual_Series_AKC_Parallel
- removed R12: 14k, Resistor_SMD:R_0805_2012Metric_Pad1.20x1.40mm_HandSolder, symbol Device:R_Small
- removed R19: 120, Resistor_SMD:R_0805_2012Metric_Pad1.20x1.40mm_HandSolder, symbol Device:R_Small
- removed R20: 1k, Resistor_SMD:R_0805_2012Metric_Pad1.20x1.40mm_HandSolder, symbol Device:R_Small
- removed R59: 100, Resistor_SMD:R_0805_2012Metric_Pad1.20x1.40mm_HandSolder, symbol Device:R_Small
- removed U2, U3: ~, Package_TO_SOT_SMD:SOT-23-5, symbol Amplifier_Operational:LMV321
- added C35, C36, C37, C38: 10u, Capacitor_SMD:C_1206_3216Metric_Pad1.33x1.80mm_HandSolder, symbol Device:C_Small
- added C39: 1u, Capacitor_SMD:C_1206_3216Metric_Pad1.33x1.80mm_HandSolder, symbol Device:C_Small
- added J34: ~, Connector_Molex:Molex_Mini-Fit_Jr_5566-04A_2x02_P4.20mm_Vertical, symbol Connector_Generic:Conn_02x02_Odd_Even
- added R23: 240, Resistor_SMD:R_0805_2012Metric_Pad1.20x1.40mm_HandSolder, symbol Device:R_Small
- added R24: 1k, Resistor_SMD:R_0805_2012Metric_Pad1.20x1.40mm_HandSolder, symbol Device:R_Small
- added U1: TLV431, Package_TO_SOT_SMD:SOT-23, symbol Reference_Voltage:TL431DBZ
- added U2: OPA333xxDBV, Package_TO_SOT_SMD:SOT-23-5, symbol Amplifier_Operational:OPA333xxDBV
- added U31: TLV1117LV33DCYR, Package_TO_SOT_SMD:SOT-223-3_TabPin2, symbol Regulator_Linear:LM1117MP-3.3
- C26, C30: value 30p -> 12p
- D18: Product Name WRB2403S-3WR2 -> WRB2405S-3WR2
- F1: footprint (none) -> Fuse_my:SMD_2410
- J6: Purpose To main connector -> +24V
- R58: value 232 -> 1k
- U4: value LM1117MP-3.3 -> TLV1117LV33DCYR
Connections:
- net +1V0: now also R23.2, R24.1; no longer R58.2
- net +24V: now also J6.2 (Pin_2), J6.4 (Pin_4), C38.1; no longer J6.3 (Pin_3)
- net +3.3V: now also U2.5 (V+)
- net +3.3VP: now also C36.2, U31.2 (VO); no longer C59.1, D18.6 (+Vo)
- net -24V: now also J6.1 (Pin_1), J6.3 (Pin_3); no longer J6.4 (Pin_4)
- net CANH: now also J34.2 (Pin_2); no longer J6.2 (Pin_2)
- net CANL: now also J34.1 (Pin_1); no longer J6.1 (Pin_1)
- net GND: now also C38.2, C39.2, U2.2 (V-)
- net GNDPWR: now also C35.1, C36.1, C37.1, R24.2, U1.3 (A), U31.1 (GND)
- net GND_CAN: now also J34.3 (Pin_3), J34.4 (Pin_4)
- net at D18.2 (Vin), L2.2: now also C39.1
- net at C15.1, R15.2: now also U2.3 (+)
- net at R18.1: now also U2.1, U2.4 (-)
- net at D18.8 (CS): now also C37.2
- new net: R23.1, R58.2, U1.1 (K), U1.2 (REF)
- new net: C35.2, C59.1, D18.6 (+Vo), U31.3 (VI)
Other:
- added sheet Voltage_measure_2 (Voltage_measure.kicad_sch)
- added sheet Voltage_measure_3 (Voltage_measure.kicad_sch)
- sheet Voltage_measure_1 ports: added VDC_SENSE; removed none
- note added: "Смещение 1В"
- note removed: "Измерение напряжения 24В"
- note removed: "Питание 1В"
- moved on the sheet: C13, C14, C15, C20, C34, C44, C59, C65, C66, C67, C68, C69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
