File: Voltage_measure.kicad_sch (KiCad schematic)
At the start: 26 parts

Commit message: VER1.0: улучшил и расставил каналы измерения напряжения
Parts:
- removed U1: ~, Package_TO_SOT_SMD:SOT-23-5, symbol Amplifier_Operational:LMV321
- added D6: TO-3216BC-MYF, LED_SMD:LED_1206_3216Metric_Pad1.42x1.75mm_HandSolder, symbol Device:LED_Small
- added D7: S1M, Diode_SMD:D_SMA_Handsoldering, symbol Device:D_Small
- added R25, R26, R27: 150k, Resistor_SMD:R_1206_3216Metric, symbol Device:R
- added U6: OPA333xxDBV, Package_TO_SOT_SMD:SOT-23-5, symbol Amplifier_Operational:OPA333xxDBV
- J3: Purpose VDC -> VDC+
Connections:
- net +3.3V: now also U6.5 (V+)
- net GND: now also U6.2 (V-)
- net at C12.1, R13.2, R21.1: now also U6.4 (-)
- net at C12.2, R10.1, R21.2: now also U6.1
- net at C1.2, R4.2, R8.2: now also U6.3 (+)
- net GNDPWR: now reaches C22.1, C23.2, C9.2, D2.3 (SHTDN), D2.4 (GND1), J7.1 (Pin_1), J7.2 (Pin_2), R9.1
- net GNDPWR: now also D7.1 (K)
- net at J3.1 (Pin_1), J3.2 (Pin_2), R1.2: now also R27.1
- new net: R26.1, R27.2
- new net: R25.1, R26.2
- new net: D6.1 (K), D7.2 (A)
- new net: D6.2 (A), R25.2
